File: electronics/waterdrop-esphome/waterdrop-esphome.kicad_pcb (KiCad board)
At the start: 4 copper layers, 64.8 x 53.3 mm, 40 parts, among them J1 12V_IN, J2 12V_OUT, J3 Comm_RO, J4 Comm_Faucet, J5 Valve, K1 G5LE-1, Q1 BC817, U1 LM2596DS-ADJ, U2 ESP32-S3-Tiny, U3 74AHCT125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

Commit message: PCB: add signature
Other:
- board text added: "waterdrop-esphome v0.1"
- board text added: "www.wasilczyk.pl"
Changed lines of the file:
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@@
 		(layer "Edge.Cuts")
+	)
+	(gr_text "waterdrop-esphome v0.1"
+		(at 137.795 114.3 90)
+		(layer "F.Cu")
+		(effects
+			(font
+				(size 1 1)
+				(thickness 0.2)
+			)
+			(justify right bottom)
+		)
+	)
+	(gr_text "www.wasilczyk.pl"
+		(at 139.7 114.3 90)
+		(layer "F.Cu")
+		(effects
+			(font
+				(size 1 1)
+				(thickness 0.2)
+			)
+			(justify right bottom)
+		)
+	)
+	(gr_text "www.wasilczyk.pl"
+		(at 171.45 85.09 0)
+		(layer "B.Cu")
+		(effects
+			(font
+				(size 0.9 0.9)
+				(thickness 0.2)
+				(bold yes)
+			)
+			(justify left bottom mirror)
+		)
 	)
 	(dimension

Commit message: Bump PCB version to 0.2
Other:
- board text added: "waterdrop-esphome v0.2"
- board text removed: "waterdrop-esphome v0.1"
Changed lines of the file:
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@@
 	(title_block
 		(title "waterdrop-esphome")
-		(date "2026-01-12")
-		(rev "0.0.1")
+		(date "2026-06-06")
+		(rev "0.2")
 		(company "Tomasz Wasilczyk")
 	)
@@
 		(layer "Edge.Cuts")
 	)
-	(gr_text "waterdrop-esphome v0.1"
+	(gr_text "waterdrop-esphome v0.2"
 		(at 137.795 114.3 90)
 		(layer "F.Cu")

Commit message: Update PCB to reflect schematic fixes
Parts:
- removed R8: 10k, Resistor_SMD:R_0805_2012Metric_Pad1.20x1.40mm_HandSolder
- C1: value 100µF/16V -> 100µF/50V; footprint Capacitor_THT:CP_Radial_D6.3mm_P2.50mm -> Capacitor_THT:CP_Radial_D8.0mm_P3.50mm
- D1: value SMAJ13A -> SMAJ30A
- D2: value B220A -> B360A
- D3: footprint Diode_SMD:D_SOD-123 -> Diode_SMD_extra:D_SOD-123_Handsoldering
- H1: value 12V_OUT_RELIEF -> 24V_OUT_RELIEF
- H3, H4: footprint MountingHole:MountingHole_4.3mm_M4 -> MountingHole:MountingHole_3.2mm_M3
- J1: value 12V_IN -> 24V_IN
- J2: value 12V_OUT -> 24V_OUT
- K1: value G5LE-1 -> G5LE-1-E DC24
- Q1: footprint Package_TO_SOT_SMD:SOT-23 -> Package_TO_SOT_SMD:SOT-23_Handsoldering
- R10, R12, R7: value 50k -> 51k
- R4: value 100k -> 47k
- moved C1 2.23 mm to (109.5, 87.0), turned to 0 degrees
- moved C2 2.21 mm to (117.6, 85.1), turned to 0 degrees
Connections:
- net +12V renamed +24V
- net /12V_IN renamed /24V_IN
- net /12V_OUT renamed /24V_OUT
- net /12V_control renamed /24V_control
Routing:
- net +5V: track 131.1 -> 122.8 mm
- net /RO_RX_HV: track 9.50 -> 6.42 mm
- net Net-(C2-Pad1): track 26.7 -> 28.3 mm
- net +24V: track 127.4 -> 128.2 mm
- net Net-(Q1-B): track 3.91 -> 3.35 mm
Other:
- board size 64.8 x 53.3 mm -> 65.4 x 53.3 mm

Commit message: Fix PCB 0.1 nits
Routing:
- net GND: track 58.2 -> 59.4 mm
- net +5V: track 122.8 -> 122.1 mm
Changed lines of the file:
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@@
 		(tags "Power Jack")
 		(property "Reference" "J1"
-			(at -9.175 5.81 180)
+			(at -9.088 6.064 180)
 			(layer "F.SilkS")
 			(effects
@@
 		(tags "Through hole angled pin header THT 1x02 2.54mm single row")
 		(property "Reference" "J5"
-			(at 1.27 -3.175 0)
+			(at 1.27 -2.5 0)
 			(layer "F.SilkS")
 			(effects
@@
 		(tags "net tie solder jumper bridged")
 		(property "Reference" "JP1"
-			(at 0 -1.8 90)
+			(at 2.5 0 180)
 			(layer "F.SilkS")
 			(effects
@@
 		(tags "Diode SMA (DO-214AC) Handsoldering")
 		(property "Reference" "D2"
-			(at 0 2.5 90)
+			(at 0 2.794 90)
 			(layer "B.SilkS")
 			(effects
@@
 		(tags "Diode SMA (DO-214AC) Handsoldering")
 		(property "Reference" "D1"
-			(at 0 -2.54 90)
+			(at 0 -2.921 90)
 			(layer "B.SilkS")
 			(effects
@@
 	)
 	(via
-		(at 113.665 123.825)
+		(at 162.56 97.79)
 		(size 1)
 		(drill 0.4)
@@
 	)
 	(via
-		(at 167.64 86.995)
+		(at 113.665 123.825)
 		(size 1)
 		(drill 0.4)
@@
 	)
 	(via
-		(at 125.73 109.855)
+		(at 167.64 86.995)
 		(size 1)
 		(drill 0.4)
@@
 	)
 	(via
-		(at 134.62 82.55)
+		(at 125.73 109.855)
 		(size 1)
 		(drill 0.4)
@@
 	)
 	(via
-		(at 167.64 99.06)
+		(at 134.62 82.55)
 		(size 1)
 		(drill 0.4)
@@
 	)
 	(via
-		(at 113.665 100.965)
+		(at 167.64 97.79)
 		(size 1)
 		(drill 0.4)
@@
 	)
 	(via
-		(at 153.035 96.52)
+		(at 113.665 100.965)
 		(size 1)
 		(drill 0.4)
@@
 	)
 	(via
-		(at 130.234354 99.119354)
+		(at 153.035 96.52)
 		(size 1)
 		(drill 0.4)
@@
 	)
 	(via
-		(at 162.56 97.798)
+		(at 130.234354 99.119354)
 		(size 1)
 		(drill 0.4)
@@
 	(segment
 		(start 167.64 99.925)
-		(end 167.64 99.06)
+		(end 167.64 97.79)
 		(width 0.8)
 		(layer "B.Cu")
@@
 	)
 	(segment
-		(start 162.56 99.925)
-		(end 162.56 97.798)
-		(width 0.8)
-		(layer "B.Cu")
-		(net 1)
-	)
-	(segment
 		(start 167.14 131.54)
 		(end 166.37 130.77)
@@
 	)
 	(segment
+		(start 162.56 99.925)
+		(end 162.56 97.79)
+		(width 0.8)
+		(layer "B.Cu")
+		(net 1)
+	)
+	(segment
 		(start 125.73 109.855)
 		(end 125.73 109.09)
@@
 	)
 	(segment
-		(start 166.37 102.44191)
-		(end 166.37 97.79)
-		(width 0.8)
-		(layer "In2.Cu")
-		(net 16)
-	)
-	(segment
-		(start 164.919 103.89291)
-		(end 164.919 119.159)
-		(width 0.8)
-		(layer "In2.Cu")
-		(net 16)
-	)
-	(segment
-		(start 166.37 88.265)
-		(end 166.37 97.79)
-		(width 0.8)
-		(layer "In2.Cu")
-		(net 16)
-	)
-	(segment
-		(start 166.37 97.79)
-		(end 165.1 97.79)
+		(start 166.37 120.61)
+		(end 164.084 118.324)
 		(width 0.8)
 		(layer "In2.Cu")
@@
 	)
 	(segment
-		(start 166.37 102.44191)
-		(end 164.919 103.89291)
-		(width 0.8)
-		(layer "In2.Cu")
-		(net 16)
-	)
-	(segment
-		(start 164.919 119.159)
-		(end 166.37 120.61)
+		(start 165.1 97.79)
+		(end 165.1 96.012)
 		(width 0.8)
 		(layer "In2.Cu")
@@
 	)
 	(segment
-		(start 164.007 96.697)
-		(end 159.208 96.697)
+		(start 165.1 96.012)
+		(end 165.1 89.535)
 		(width 0.8)
 		(layer "In2.Cu")
@@
 	)
 	(segment
-		(start 165.1 97.79)
-		(end 164.007 96.697)
+		(start 158.115 97.79)
+		(end 159.893 96.012)
 		(width 0.8)
 		(layer "In2.Cu")
@@
 	)
 	(segment
-		(start 159.208 96.697)
-		(end 158.115 97.79)
+		(start 164.084 118.324)
+		(end 164.084 98.806)
+		(width 0.8)
+		(layer "In2.Cu")
+		(net 16)
+	)
+	(segment
+		(start 159.893 96.012)
+		(end 165.1 96.012)
 		(width 0.8)
 		(layer "In2.Cu")
@@
 	)
 	(segment
+		(start 165.1 89.535)
+		(end 166.37 88.265)
+		(width 0.8)
+		(layer "In2.Cu")
+		(net 16)
+	)
+	(segment
 		(start 137.607788 86.991)
 		(end 123.829 86.991)
 		(width 0.8)
 		(layer "In2.Cu")
+		(net 16)
+	)
+	(segment
+		(start 164.084 98.806)
+		(end 165.1 97.79)
+		(width 0.8)
+		(layer "In2.Cu")

Commit message: Bump PCB version to 1.0 and firmware to 1.0.0
Other:
- board text added: "waterdrop-esphome v1.0"
- board text removed: "waterdrop-esphome v0.2"
Changed lines of the file:
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@@
 	(title_block
 		(title "waterdrop-esphome")
-		(date "2026-06-06")
-		(rev "0.2")
+		(date "2026-06-27")
+		(rev "1.0")
 		(company "Tomasz Wasilczyk")
 	)
@@
 		(layer "Edge.Cuts")
 	)
-	(gr_text "waterdrop-esphome v0.2"
+	(gr_text "waterdrop-esphome v1.0"
 		(at 137.795 114.3 90)
 		(layer "F.Cu")
