File: electronics/waterdrop-esphome/waterdrop-esphome.kicad_sch (KiCad schematic)
At the start: 26 parts, among them J1 24V_IN, J2 24V_OUT, J3 Comm_RO, J4 Comm_Faucet, J5 Valve, K1 G5LE-1-E DC24, Q1 BC817, U2 ESP32-S3-Tiny, U3 74AHCT125, U4 TB67H450A

Commit message: Update footprints: D3 and Q1 hand soldering, C1 size
Parts:
- D3: footprint Diode_SMD:D_SOD-123 -> Diode_SMD_extra:D_SOD-123_Handsoldering
- Q1: footprint Package_TO_SOT_SMD:SOT-23 -> Package_TO_SOT_SMD:SOT-23_Handsoldering
Changed lines of the file:
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@@
 			)
 		)
-		(property "Footprint" "Diode_SMD:D_SOD-123"
+		(property "Footprint" "Diode_SMD_extra:D_SOD-123_Handsoldering"
 			(at 95.25 48.26 0)
 			(effects
@@
 			)
 		)
-		(property "Footprint" "Package_TO_SOT_SMD:SOT-23"
+		(property "Footprint" "Package_TO_SOT_SMD:SOT-23_Handsoldering"
 			(at 92.71 65.405 0)
 			(effects
